Commit message: Implemented chaser-target scenario in rviz

File: astrobee_description/models/chaser/model.urdf.xacro (robot description, xacro)
@@ -16,5 +16,5 @@
 <!-- implied. See the License for the specific language governing            -->
 <!-- permissions and limitations under the License.                          -->
-<robot name="astrobee" xmlns:xacro="http://www.ros.org/wiki/xacro">
+<robot name="chaser" xmlns:xacro="http://www.ros.org/wiki/xacro">
   <!-- OPTIONS -->
   <!-- <xacro:property name="world" value="$(arg world)"/>
@@ -28,5 +28,5 @@
   </xacro:if> -->
   <!-- BASE GEOMETRY -->
- <link name="base_link">
+ <link name="chaser/base_link">
     <self_collide>false</self_collide>
     <!-- body -->
@@ -95,5 +95,5 @@
   </link>
   <!-- This is a workaround for KDL -->
-  <link name="inertial_link">
+  <link name="chaser/inertial_link">
     <self_collide>false</self_collide>
     <inertial>
@@ -105,6 +105,6 @@
   <joint name="inertial_joint" type="fixed">
     <origin xyz="0 0 0" rpy="0 0 0" />
-    <parent link="base_link" />
-    <child link="inertial_link" />
+    <parent link="chaser/base_link" />
+    <child link="chaser/inertial_link" />
   </joint>
 </robot>

File: astrobee_description/models/target/model.urdf.xacro (robot description, xacro)
@@ -16,5 +16,5 @@
 <!-- implied. See the License for the specific language governing            -->
 <!-- permissions and limitations under the License.                          -->
-<robot name="astrobee" xmlns:xacro="http://www.ros.org/wiki/xacro">
+<robot name="target" xmlns:xacro="http://www.ros.org/wiki/xacro">
   <!-- OPTIONS -->
   <!-- <xacro:property name="world" value="$(arg world)"/>
@@ -28,5 +28,5 @@
   </xacro:if> -->
   <!-- BASE GEOMETRY -->
- <link name="base_link">
+ <link name="target/base_link">
     <self_collide>false</self_collide>
     <!-- body -->
@@ -95,5 +95,5 @@
   </link>
   <!-- This is a workaround for KDL -->
-  <link name="inertial_link">
+  <link name="target/inertial_link">
     <self_collide>false</self_collide>
     <inertial>
@@ -105,6 +105,6 @@
   <joint name="inertial_joint" type="fixed">
     <origin xyz="0 0 0" rpy="0 0 0" />
-    <parent link="base_link" />
-    <child link="inertial_link" />
+    <parent link="target/base_link" />
+    <child link="target/inertial_link" />
   </joint>
 </robot>
